File: HW/Relay/Eagle/relay.sch (EAGLE design)
At the start: 45 parts, among them IC2 DS18B20, J1 284513-2, J2 284513-2, J3 284513-3, K2 CQ1-12V, M1 WIRELESS-NRF24L01, T1 BC847, U3 MCP16311

Commit message: Add files via upload
Parts:
- removed J1, J2: 284513-2, 284513-2:284513-2
- removed J3: 284513-3, 284513-3:284513-3
- added R2: 10K, rcl:R-US_M2012
- added X1: MC3-G, con-phoenix-381_l:MC3-G
- added X2, X3: MC2-G, con-phoenix-381_l:MC2-G
Connections:
- net BUTTON_CONTROL: now also R2.1, SJR2.GPIO2; no longer SJR2.GPIO4
- net C: now also X1.2.SK; no longer J3.2
- net GND: now also X2.2.SK; no longer J1.2
- net N$11: now also X3.1.SK; no longer J2.2
- net N$12: now also X3.2.SK; no longer J2.1
- net NC: now also X1.1.SK; no longer J3.3
- net NO: now also X1.3.SK; no longer J3.1
- net RF_CE: now also SJR2.GPIO4; no longer SJR2.GPIO2
- net RF_IRQ: no longer SJR2.GPIO0
- net VCC: now also R2.2
- net VIN: now also X2.1.SK; no longer J1.1
Changed lines of the file:
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@@
 <part name="M1" library="diy-modules" deviceset="WIRELESS-NRF24L01" device=""/>
 <part name="GND4" library="supply1" library_urn="urn:adsk.eagle:library:371" deviceset="GND" device=""/>
-<part name="J1" library="284513-2" deviceset="284513-2" device=""/>
-<part name="J2" library="284513-2" deviceset="284513-2" device=""/>
-<part name="J3" library="284513-3" deviceset="284513-3" device=""/>
+<part name="X1" library="con-phoenix-381_l" deviceset="MC3-G" device=""/>
+<part name="X2" library="con-phoenix-381_l" deviceset="MC2-G" device=""/>
+<part name="X3" library="con-phoenix-381_l" deviceset="MC2-G" device=""/>
+<part name="R2" library="rcl" library_urn="urn:adsk.eagle:library:334" deviceset="R-US_" device="M2012" package3d_urn="urn:adsk.eagle:package:23561/2" value="10K"/>
+<part name="SUPPLY2" library="SparkFun-Aesthetics" deviceset="VCC" device=""/>
 </parts>
 <sheets>
@@
 <attribute name="VALUE" x="254" y="149.86" size="1.778" layer="96" rot="R270"/>
 </instance>
-<instance part="J1" gate="G$1" x="200.66" y="251.46" smashed="yes">
-<attribute name="NAME" x="195.08" y="256.54" size="1.778" layer="95"/>
-<attribute name="VALUE" x="195.58" y="246.38" size="1.778" layer="96"/>
-</instance>
-<instance part="J2" gate="G$1" x="116.84" y="76.2" smashed="yes" rot="R180">
-<attribute name="NAME" x="122.42" y="71.12" size="1.778" layer="95" rot="R180"/>
-<attribute name="VALUE" x="121.92" y="81.28" size="1.778" layer="96" rot="R180"/>
-</instance>
-<instance part="J3" gate="G$1" x="411.48" y="203.2" smashed="yes" rot="R180">
-<attribute name="NAME" x="414.02503125" y="197.34641875" size="1.78151875" layer="95" rot="R180"/>
-<attribute name="VALUE" x="414.02198125" y="210.825940625" size="1.779390625" layer="96" rot="R180"/>
+<instance part="X1" gate=".1" x="381" y="231.14" smashed="yes">
+<attribute name="VALUE" x="375.92" y="227.8528" size="1.524" layer="96"/>
+<attribute name="NAME" x="367.03" y="230.505" size="1.524" layer="95"/>
+</instance>
+<instance part="X1" gate=".2" x="381" y="226.06" smashed="yes">
+<attribute name="VALUE" x="375.92" y="222.7728" size="1.524" layer="96"/>
+<attribute name="NAME" x="367.03" y="225.425" size="1.524" layer="95"/>
+</instance>
+<instance part="X1" gate=".3" x="381" y="220.98" smashed="yes">
+<attribute name="VALUE" x="375.92" y="217.6928" size="1.524" layer="96"/>
+<attribute name="NAME" x="367.03" y="220.345" size="1.524" layer="95"/>
+</instance>
+<instance part="X2" gate=".1" x="203.2" y="254" smashed="yes" rot="R180">
+<attribute name="VALUE" x="208.28" y="257.2872" size="1.524" layer="96" rot="R180"/>
+<attribute name="NAME" x="217.17" y="254.635" size="1.524" layer="95" rot="R180"/>
+</instance>
+<instance part="X2" gate=".2" x="203.2" y="248.92" smashed="yes" rot="R180">
+<attribute name="VALUE" x="208.28" y="252.2072" size="1.524" layer="96" rot="R180"/>
+<attribute name="NAME" x="217.17" y="249.555" size="1.524" layer="95" rot="R180"/>
+</instance>
+<instance part="X3" gate=".1" x="119.38" y="76.2" smashed="yes">
+<attribute name="VALUE" x="114.3" y="72.9128" size="1.524" layer="96"/>
+<attribute name="NAME" x="105.41" y="75.565" size="1.524" layer="95"/>
+</instance>
+<instance part="X3" gate=".2" x="119.38" y="71.12" smashed="yes">
+<attribute name="VALUE" x="114.3" y="67.8328" size="1.524" layer="96"/>
+<attribute name="NAME" x="105.41" y="70.485" size="1.524" layer="95"/>
+</instance>
+<instance part="R2" gate="G$1" x="170.18" y="175.26" smashed="yes" rot="R90">
+<attribute name="NAME" x="168.6814" y="171.45" size="1.778" layer="95" rot="R90"/>
+<attribute name="VALUE" x="173.482" y="171.45" size="1.778" layer="96" rot="R90"/>
+</instance>
+<instance part="SUPPLY2" gate="G$1" x="170.18" y="190.5" smashed="yes">
+<attribute name="VALUE" x="169.164" y="194.056" size="1.778" layer="96"/>
 </instance>
 </instances>
@@
 </segment>
 <segment>
-<pinref part="GND13" gate="1" pin="GND"/>
-<wire x1="189.484" y1="249.936" x2="180.594" y2="249.936" width="0.1524" layer="91"/>
-<wire x1="180.594" y1="249.936" x2="180.594" y2="229.616" width="0.1524" layer="91"/>
-<pinref part="J1" gate="G$1" pin="2"/>
-<wire x1="190.5" y1="251.46" x2="189.484" y2="251.46" width="0.1524" layer="91"/>
-<wire x1="189.484" y1="251.46" x2="189.484" y2="249.936" width="0.1524" layer="91"/>
-</segment>
-<segment>
 <pinref part="M1" gate="G$1" pin="GND"/>
 <wire x1="274.32" y1="147.32" x2="259.08" y2="147.32" width="0.1524" layer="91"/>
 <pinref part="GND4" gate="1" pin="GND"/>
+</segment>
+<segment>
+<pinref part="GND13" gate="1" pin="GND"/>
+<pinref part="X2" gate=".2" pin="SK"/>
+<wire x1="180.594" y1="229.616" x2="180.594" y2="248.92" width="0.1524" layer="91"/>
+<wire x1="180.594" y1="248.92" x2="195.58" y2="248.92" width="0.1524" layer="91"/>
 </segment>
 </net>
@@
 <wire x1="172.72" y1="76.2" x2="172.72" y2="86.36" width="0.1524" layer="91"/>
 </segment>
+<segment>
+<pinref part="R2" gate="G$1" pin="2"/>
+<wire x1="170.18" y1="180.34" x2="170.18" y2="190.5" width="0.1524" layer="91"/>
+<pinref part="SUPPLY2" gate="G$1" pin="VCC"/>
+</segment>
 </net>
 <net name="VIN" class="0">
@@
 <wire x1="180.34" y1="255.016" x2="180.34" y2="264.16" width="0.1524" layer="91"/>
 <label x="180.34" y="264.16" size="1.27" layer="95" rot="R90" xref="yes"/>
-<pinref part="J1" gate="G$1" pin="1"/>
-<wire x1="190.5" y1="254" x2="190.5" y2="255.016" width="0.1524" layer="91"/>
 <wire x1="190.5" y1="255.016" x2="180.34" y2="255.016" width="0.1524" layer="91"/>
+<pinref part="X2" gate=".1" pin="SK"/>
+<wire x1="190.5" y1="255.016" x2="190.5" y2="254" width="0.1524" layer="91"/>
+<wire x1="190.5" y1="254" x2="195.58" y2="254" width="0.1524" layer="91"/>
 </segment>
 </net>
@@
 </segment>
 <segment>
-<pinref part="J3" gate="G$1" pin="3"/>
-<wire x1="401.32" y1="205.74" x2="393.7" y2="205.74" width="0.1524" layer="91"/>
-<label x="393.7" y="205.74" size="1.016" layer="95" rot="R180" xref="yes"/>
+<pinref part="X1" gate=".1" pin="SK"/>
+<wire x1="388.62" y1="231.14" x2="396.24" y2="231.14" width="0.1524" layer="91"/>
+<label x="396.24" y="231.14" size="1.778" layer="95" xref="yes"/>
 </segment>
 </net>
@@
 </segment>
 <segment>
-<pinref part="J3" gate="G$1" pin="2"/>
-<wire x1="401.32" y1="203.2" x2="393.7" y2="203.2" width="0.1524" layer="91"/>
-<label x="393.7" y="203.2" size="1.016" layer="95" rot="R180" xref="yes"/>
+<pinref part="X1" gate=".2" pin="SK"/>
+<wire x1="388.62" y1="226.06" x2="396.24" y2="226.06" width="0.1524" layer="91"/>
+<label x="396.24" y="226.06" size="1.778" layer="95" xref="yes"/>
 </segment>
 </net>
@@
 </segment>
 <segment>
-<pinref part="J3" gate="G$1" pin="1"/>
-<wire x1="401.32" y1="200.66" x2="393.7" y2="200.66" width="0.1524" layer="91"/>
-<label x="393.7" y="200.66" size="1.016" layer="95" rot="R180" xref="yes"/>
+<pinref part="X1" gate=".3" pin="SK"/>
+<wire x1="388.62" y1="220.98" x2="396.24" y2="220.98" width="0.1524" layer="91"/>
+<label x="396.24" y="220.98" size="1.778" layer="95" xref="yes"/>
 </segment>
 </net>
@@
 </segment>
 <segment>
-<pinref part="SJR2" gate="G$1" pin="GPIO2"/>
-<wire x1="149.86" y1="142.24" x2="157.48" y2="142.24" width="0.1016" layer="91"/>
-<label x="157.48" y="142.24" size="1.016" layer="95" xref="yes"/>
+<pinref part="SJR2" gate="G$1" pin="GPIO4"/>
+<wire x1="149.86" y1="147.32" x2="172.72" y2="147.32" width="0.1524" layer="91"/>
+<label x="172.72" y="147.32" size="1.778" layer="95" xref="yes"/>
 </segment>
 </net>
@@
 <pinref part="R11" gate="G$1" pin="1"/>
 <wire x1="147.32" y1="71.12" x2="127" y2="71.12" width="0.1524" layer="91"/>
-<pinref part="J2" gate="G$1" pin="1"/>
-<wire x1="127" y1="71.12" x2="127" y2="73.66" width="0.1524" layer="91"/>
+<pinref part="X3" gate=".2" pin="SK"/>
 </segment>
 </net>
@@
 <pinref part="R5" gate="G$1" pin="1"/>
 <wire x1="137.16" y1="76.2" x2="127" y2="76.2" width="0.1524" layer="91"/>
-<pinref part="J2" gate="G$1" pin="2"/>
+<pinref part="X3" gate=".1" pin="SK"/>
 </segment>
 </net>
@@
 <label x="259.08" y="129.54" size="1.016" layer="95" rot="R180" xref="yes"/>
 </segment>
-<segment>
-<pinref part="SJR2" gate="G$1" pin="GPIO0"/>
-<wire x1="149.86" y1="144.78" x2="157.48" y2="144.78" width="0.1524" layer="91"/>
-<label x="157.48" y="144.78" size="1.016" layer="95" xref="yes"/>
-</segment>
 </net>
 <net name="BUTTON_CONTROL" class="0">
-<segment>
-<pinref part="SJR2" gate="G$1" pin="GPIO4"/>
-<wire x1="149.86" y1="147.32" x2="172.72" y2="147.32" width="0.1524" layer="91"/>
-<label x="172.72" y="147.32" size="1.778" layer="95" xref="yes"/>
-</segment>
 <segment>
 <pinref part="R12" gate="G$1" pin="2"/>
@@
 <label x="182.88" y="71.12" size="1.778" layer="95" xref="yes"/>
 </segment>
-</net>
+<segment>
+<pinref part="SJR2" gate="G$1" pin="GPIO2"/>
+<wire x1="149.86" y1="142.24" x2="170.18" y2="142.24" width="0.1016" layer="91"/>
+<label x="177.8" y="142.24" size="1.778" layer="95" xref="yes"/>
+<pinref part="R2" gate="G$1" pin="1"/>
+<wire x1="170.18" y1="142.24" x2="177.8" y2="142.24" width="0.1016" layer="91"/>
+<wire x1="170.434" y1="170.18" x2="170.18" y2="170.18" width="0.1524" layer="91"/>
+<wire x1="170.18" y1="170.18" x2="170.18" y2="142.24" width="0.1524" layer="91"/>
+<junction x="170.18" y="170.18"/>
+<junction x="170.18" y="142.24"/>
+</segment>
+</net>

Commit message: Add files via upload
Parts:
- added R3: 10K, rcl:R-US_M2012
Connections:
- net GND: now also R3.1
- net RF_CSN: now also R3.2
Changed lines of the file:
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@@
 <part name="R2" library="rcl" library_urn="urn:adsk.eagle:library:334" deviceset="R-US_" device="M2012" package3d_urn="urn:adsk.eagle:package:23561/2" value="10K"/>
 <part name="SUPPLY2" library="SparkFun-Aesthetics" deviceset="VCC" device=""/>
+<part name="GND10" library="supply1" library_urn="urn:adsk.eagle:library:371" deviceset="GND" device=""/>
+<part name="R3" library="rcl" library_urn="urn:adsk.eagle:library:334" deviceset="R-US_" device="M2012" package3d_urn="urn:adsk.eagle:package:23561/2" value="10K"/>
 </parts>
 <sheets>
@@
 <attribute name="VALUE" x="169.164" y="194.056" size="1.778" layer="96"/>
 </instance>
+<instance part="GND10" gate="1" x="156.718" y="112.522" smashed="yes" rot="MR0">
+<attribute name="VALUE" x="159.258" y="109.982" size="1.778" layer="96" rot="MR0"/>
+</instance>
+<instance part="R3" gate="G$1" x="153.924" y="124.968" smashed="yes" rot="R90">
+<attribute name="NAME" x="152.4254" y="121.158" size="1.778" layer="95" rot="R90"/>
+<attribute name="VALUE" x="157.226" y="121.158" size="1.778" layer="96" rot="R90"/>
+</instance>
 </instances>
 <busses>
@@
 <wire x1="180.594" y1="229.616" x2="180.594" y2="248.92" width="0.1524" layer="91"/>
 <wire x1="180.594" y1="248.92" x2="195.58" y2="248.92" width="0.1524" layer="91"/>
+</segment>
+<segment>
+<pinref part="R3" gate="G$1" pin="1"/>
+<pinref part="GND10" gate="1" pin="GND"/>
+<wire x1="153.924" y1="119.888" x2="153.924" y2="115.062" width="0.1524" layer="91"/>
+<wire x1="153.924" y1="115.062" x2="156.718" y2="115.062" width="0.1524" layer="91"/>
 </segment>
 </net>
@@
 <segment>
 <pinref part="SJR2" gate="G$1" pin="GPIO15"/>
-<wire x1="149.86" y1="139.7" x2="157.48" y2="139.7" width="0.1524" layer="91"/>
+<wire x1="149.86" y1="139.7" x2="153.924" y2="139.7" width="0.1524" layer="91"/>
 <label x="157.48" y="139.7" size="1.016" layer="95" xref="yes"/>
-</segment>
-</net>
+<wire x1="153.924" y1="139.7" x2="157.48" y2="139.7" width="0.1524" layer="91"/>
+<wire x1="153.924" y1="139.7" x2="153.924" y2="130.048" width="0.1524" layer="91"/>
+<junction x="153.924" y="139.7"/>
+<pinref part="R3" gate="G$1" pin="2"/>
+<wire x1="153.924" y1="130.048" x2="153.924" y2="129.54" width="0.1524" layer="91"/>
+<junction x="153.924" y="130.048"/>
+</segment>
+</net>
