File: HW/Reader/Eagle/door_lock_v1.2.sch (EAGLE design)
At the start: 47 parts, among them Q4 BC817, U1 MCP16311, U2 ESP8266-12E

Commit message: Minor improvements on schematic
Parts:
- D7: value 1A/40V/500mV -> SS14
- LED1: device adafruit:LEDIRL80A -> led:LED3MM
- R1: value 200 -> 220
Connections:
- net BUZZ_TO_ESP renamed BUZZER
- net IR_REC_DATA renamed IR_RX
- net PROG_IR_TR renamed IR_TX
Other:
- note added: "ESP-12 based WiFi Mifare Reader"
- note added: "ESP12E Module"
- note added: "Programming Socket"
- note added: "TODO for PCB : - Check VIN connector - Check Buzzer - Check IR Sensor - Check MFRC Module"
- note removed: "ESP-12 non-wired communication between door relay & RFID Reader"
- note removed: "ESP12E_IC"
- note removed: "Programming_Output"
- moved on the sheet: C1, C10, C11, C12, C2, C20, C3, C4, C5, C6, C7, C8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
